Commit message: Created core URDF

File: description/gazebo_control.xacro (robot description, xacro)
@@ -6,6 +6,6 @@
            <left_joint>left_wheel_joint</left_joint>
            <right_joint>right_wheel_joint</right_joint>
-           <wheel_separation>0.35</wheel_separation>
-           <wheel_diameter>0.1</wheel_diameter>
+           <wheel_separation>0.415</wheel_separation>
+           <wheel_diameter>0.045</wheel_diameter>
            <!--Limits-->
            <max_wheel_torque>200</max_wheel_torque>

File: description/lidar.xacro (robot description, xacro)
@@ -2,7 +2,7 @@
 <robot xmlns:xacro="http://www.ros.org/wiki/xacro"  >
     <joint name="laser_joint" type="fixed">
-       <parent link="chassis"/>
+       <parent link="lidar_mount"/>
        <child link="laser_frame"/>
-       <origin xyz="0.1 0 0.175" rpy="0 0 0"/>
+       <origin xyz="0 0 0.035" rpy="0 0 0"/>
     </joint>
     <link name="laser_frame">

File: description/robot.urdf.xacro (robot description, xacro)
@@ -2,5 +2,7 @@
 <robot xmlns:xacro="http://www.ros.org/wiki/xacro"  name="robot">
       <xacro:include filename="robot_core.xacro" />
-      <xacro:include filename="gazebo_control.xacro" />
+      <!-- <xacro:include filename="gazebo_control.xacro" /> -->
       <xacro:include filename="lidar.xacro" />
+      <xacro:include filename="camera.xacro" />
+      <xacro:include filename="ros2_control.xacro" />
 </robot>

File: description/robot_core.xacro (robot description, xacro)
@@ -17,112 +17,410 @@
          <color rgba="1 0 0 1" />
     </material>
-    <!-- BASE LINK -->
+<!-- BASE LINK -->
     <link name="base_link">
     </link>
-    <!-- CHASSIS LINK -->
-    <joint name="chassis_joint" type="fixed">
-          <parent link="base_link" />
-          <child link="chassis" />
-          <origin xyz="-0.1 0 0" />
-    </joint>
-    <link name="chassis">
-          <visual>
-            <origin xyz="0.15 0 0.075" />
-            <geometry>
-               <box size="0.3 0.3 0.15" />
-            </geometry>
-            <material name="white" />
-          </visual>
-          <collision>
-            <origin xyz="0.15 0 0.075" />
-            <geometry>
-               <box size="0.3 0.3 0.15" />
-            </geometry>
-          </collision>
-          <xacro:inertial_box mass="0.5" x="0.3" y="0.3" z="0.15">
-              <origin xyz="0.15 0 0.075" rpy="0 0 0" />
-          </xacro:inertial_box>
-    </link>
-    <gazebo reference="chassis">
-        <material>Gazebo/White</material>
-    </gazebo>
-    <!-- LEFT WHEEL LINK -->
-    <joint name="left_wheel_joint" type="continuous">
-           <parent link="base_link" />
-           <child link="left_wheel" />
-           <origin xyz="0 0.175 0" rpy="-${pi/2} 0 0" />
-           <axis xyz="0 0 1" />
-    </joint>
-    <link name="left_wheel">
-        <visual>
-           <geometry>
-             <cylinder radius="0.05" length="0.04" />
-           </geometry>
-           <material name="blue" />
-        </visual>
-        <collision>
-           <geometry>
-             <cylinder radius="0.05" length="0.04" />
-           </geometry>
-        </collision>
-        <xacro:inertial_cylinder mass="0.1" length="0.04" radius="0.05">
-              <origin xyz="0 0 0" rpy="0 0 0" />
-        </xacro:inertial_cylinder>
-    </link>
-    <gazebo reference="left_wheel">
-        <material>Gazebo/Blue</material>
-    </gazebo>
-    <!-- RIGHT WHEEL LINK -->
-    <joint name="right_wheel_joint" type="continuous">
-           <parent link="base_link" />
-           <child link="right_wheel" />
-           <origin xyz="0 -0.175 0" rpy="${pi/2} 0 0" />
-           <axis xyz="0 0 -1" />
-    </joint>
-    <link name="right_wheel">
-        <visual>
-           <geometry>
-             <cylinder radius="0.05" length="0.04" />
-           </geometry>
-           <material name="blue" />
-        </visual>
-        <collision>
-           <geometry>
-             <cylinder radius="0.05" length="0.04" />
-           </geometry>
-        </collision>
-        <xacro:inertial_cylinder mass="0.1" length="0.04" radius="0.05">
-              <origin xyz="0 0 0" rpy="0 0 0" />
-        </xacro:inertial_cylinder>
-    </link>
-    <gazebo reference="right_wheel">
-        <material>Gazebo/Blue</material>
-    </gazebo>
-    <!-- CASTER WHEEL LINK -->
-    <joint name="caster_wheel_joint" type="fixed">
-        <parent link="chassis" />
-        <child link="caster_wheel" />
-        <origin xyz="0.24 0 0" />
-    </joint>
-    <link name="caster_wheel">
-        <visual>
-            <geometry>
-              <sphere radius="0.05" />
-            </geometry>
-            <material name="black" />
-        </visual>
-        <collision>
-            <geometry>
-              <sphere radius="0.05" />
-            </geometry>
-        </collision>
-        <xacro:inertial_sphere mass="0.1" radius="0.05">
-            <origin xyz="0 0 0" rpy="0 0 0" />
-        </xacro:inertial_sphere>
-    </link>
-    <gazebo reference="caster_wheel">
-        <material>Gazebo/Black</material>
-        <mu1 value="0.001"/>
-        <mu2 value="0.001"/>
-    </gazebo>
+<!-- LOWER BODY -->
+<joint name="lower_body_joint" type="fixed">
+    <parent link="base_link"/>
+    <child link="lower_body"/>
+    <origin xyz="0 0 0"/>
+</joint>
+<link name="lower_body">
+    <visual>
+        <origin xyz="0 0 0.0075"/>
+        <geometry>
+            <box size="0.45 0.40 0.015"/>
+        </geometry>
+        <material name="white"/>
+    </visual>
+    <collision>
+        <origin xyz="0 0 0.0075"/>
+        <geometry>
+            <box size="0.45 0.40 0.015"/>
+        </geometry>
+    </collision>
+    <xacro:inertial_box
+        mass="1.0"
+        x="0.45"
+        y="0.40"
+        z="0.015">
+        <origin xyz="0 0 0.0075"/>
+    </xacro:inertial_box>
+</link>
+<gazebo reference="lower_body">
+    <material>Gazebo/White</material>
+</gazebo>
+<!--MIDDLE BODY-->
+<joint name="middle_body_joint" type="fixed">
+    <parent link="lower_body"/>
+    <child link="middle_body"/>
+    <origin xyz="-0.08 0 0.0775"/>
+</joint>
+<link name="middle_body">
+    <visual>
+        <geometry>
+            <box size="0.29 0.40 0.14"/>
+        </geometry>
+        <material name="white"/>
+    </visual>
+    <collision>
+        <geometry>
+            <box size="0.29 0.40 0.14"/>
+        </geometry>
+    </collision>
+    <xacro:inertial_box
+        mass="2.0"
+        x="0.29"
+        y="0.40"
+        z="0.14">
+        <origin xyz="0 0 0"/>
+    </xacro:inertial_box>
+</link>
+<gazebo reference="middle_body">
+    <material>Gazebo/White</material>
+</gazebo>
+<!--UPPER BODY-->
+<joint name="upper_body_joint" type="fixed">
+    <parent link="middle_body"/>
+    <child link="upper_body"/>
+    <origin xyz="0.08 0 0.0775"/>
+</joint>
+<link name="upper_body">
+    <visual>
+        <geometry>
+            <box size="0.45 0.40 0.015"/>
+        </geometry>
+        <material name="white"/>
+    </visual>
+    <collision>
+        <geometry>
+            <box size="0.45 0.40 0.015"/>
+        </geometry>
+    </collision>
+    <xacro:inertial_box
+        mass="1.0"
+        x="0.45"
+        y="0.40"
+        z="0.015">
+        <origin xyz="0 0 0"/>
+    </xacro:inertial_box>
+</link>
+<gazebo reference="upper_body">
+    <material>Gazebo/White</material>
+</gazebo>
+<!--LIDAR MOUNT-->
+<joint name="lidar_mount_joint" type="fixed">
+    <parent link="lower_body"/>
+    <child link="lidar_mount"/>
+    <origin xyz="0.170 0 0.040"/>
+</joint>
+<link name="lidar_mount">
+    <visual>
+        <geometry>
+            <box size="0.07 0.06 0.05"/>
+        </geometry>
+        <material name="black"/>
+    </visual>
+    <collision>
+        <geometry>
+            <box size="0.07 0.06 0.05"/>
+        </geometry>
+    </collision>
+    <xacro:inertial_box
+        mass="0.20"
+        x="0.07"
+        y="0.06"
+        z="0.05">
+        <origin xyz="0 0 0"/>
+    </xacro:inertial_box>
+</link>
+<gazebo reference="lidar_mount">
+    <material>Gazebo/Black</material>
+</gazebo>
+<!--front_left_pillar_joint-->
+<joint name="front_left_pillar_joint" type="fixed">
+    <parent link="lower_body"/>
+    <child link="front_left_pillar"/>
+    <origin xyz="0.18 0.177 0.085"/>
+</joint>
+<link name="front_left_pillar">
+    <visual>
+        <geometry>
+            <box size="0.03 0.016 0.14"/>
+        </geometry>
+        <material name="orange"/>
+    </visual>
+    <collision>
+        <geometry>
+            <box size="0.03 0.016 0.14"/>
+        </geometry>
+    </collision>
+    <xacro:inertial_box
+        mass="0.15"
+        x="0.03"
+        y="0.016"
+        z="0.14">
+        <origin xyz="0 0 0"/>
+    </xacro:inertial_box>
+</link>
+<gazebo reference="front_left_pillar">
+    <material>Gazebo/Orange</material>
+</gazebo>
+<!--front_right_pillar_joint-->
+<joint name="front_right_pillar_joint" type="fixed">
+    <parent link="lower_body"/>
+    <child link="front_right_pillar"/>
+    <origin xyz="0.18 -0.177 0.085"/>
+</joint>
+<link name="front_right_pillar">
+    <visual>
+        <geometry>
+            <box size="0.03 0.016 0.14"/>
+        </geometry>
+        <material name="orange"/>
+    </visual>
+    <collision>
+        <geometry>
+            <box size="0.03 0.016 0.14"/>
+        </geometry>
+    </collision>
+    <xacro:inertial_box
+        mass="0.15"
+        x="0.03"
+        y="0.016"
+        z="0.14">
+        <origin xyz="0 0 0"/>
+    </xacro:inertial_box>
+</link>
+<gazebo reference="front_right_pillar">
+    <material>Gazebo/Orange</material>
+</gazebo>
+<!-- LEFT MOTOR -->
+<joint name="left_motor_joint" type="fixed">
+    <parent link="lower_body"/>
+    <child link="left_motor"/>
+    <origin xyz="0 0.1725 -0.037"/>
+</joint>
+<link name="left_motor">
+    <visual>
+        <origin xyz="0 0 0"/>
+        <geometry>
+            <box size="0.14 0.055 0.074"/>
+        </geometry>
+        <material name="black"/>
+    </visual>
+    <collision>
+        <origin xyz="0 0 0"/>
+        <geometry>
+            <box size="0.14 0.055 0.074"/>
+        </geometry>
+    </collision>
+    <xacro:inertial_box
+        mass="0.5"
+        x="0.14"
+        y="0.055"
+        z="0.074">
+        <origin xyz="0 0 0"/>
+    </xacro:inertial_box>
+</link>
+<gazebo reference="left_motor">
+    <material>Gazebo/Black</material>
+</gazebo>
+<!-- RIGHT MOTOR -->
+<joint name="right_motor_joint" type="fixed">
+    <parent link="lower_body"/>
+    <child link="right_motor"/>
+    <origin xyz="0 -0.1725 -0.037"/>
+</joint>
+<link name="right_motor">
+    <visual>
+        <origin xyz="0 0 0"/>
+        <geometry>
+            <box size="0.14 0.055 0.074"/>
+        </geometry>
+        <material name="black"/>
+    </visual>
+    <collision>
+        <origin xyz="0 0 0"/>
+        <geometry>
+            <box size="0.14 0.055 0.074"/>
+        </geometry>
+    </collision>
+    <xacro:inertial_box
+        mass="0.5"
+        x="0.14"
+        y="0.055"
+        z="0.074">
+        <origin xyz="0 0 0"/>
+    </xacro:inertial_box>
+</link>
+<gazebo reference="right_motor">
+    <material>Gazebo/Black</material>
+</gazebo>
+<!-- LEFT WHEEL-->
+<joint name="left_wheel_joint" type="continuous">
+    <parent link="base_link"/>
+    <child link="left_wheel"/>
+    <origin xyz="0 0.2075 -0.05" rpy="-${pi/2} 0 0"/>
+    <axis xyz="0 0 1"/>
+</joint>
+<link name="left_wheel">
+    <visual>
+        <geometry>
+            <cylinder radius="0.05" length="0.015"/>
+        </geometry>
+        <material name="blue"/>
+    </visual>
+    <collision>
+        <geometry>
+            <cylinder radius="0.047" length="0.015"/>
+        </geometry>
+    </collision>
+    <xacro:inertial_cylinder
+        mass="0.25"
+        radius="0.05"
+        length="0.015">
+        <origin xyz="0 0 0"/>
+    </xacro:inertial_cylinder>
+</link>
+<gazebo reference="left_wheel">
+    <material>Gazebo/Blue</material>
+</gazebo>
+<!-- RIGHT WHEEL -->
+<joint name="right_wheel_joint" type="continuous">
+    <parent link="base_link"/>
+    <child link="right_wheel"/>
+    <origin xyz="0 -0.2075 -0.05" rpy="${pi/2} 0 0"/>
+    <axis xyz="0 0 -1"/>
+</joint>
+<link name="right_wheel">
+    <visual>
+        <geometry>
+            <cylinder radius="0.05" length="0.015"/>
+        </geometry>
+        <material name="blue"/>
+    </visual>
+    <collision>
+        <geometry>
+            <cylinder radius="0.05" length="0.015"/>
+        </geometry>
+    </collision>
+    <xacro:inertial_cylinder
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