Commit message: Created core URDF

File: description/robot.urdf.xacro (robot description, xacro)
@@ -1,8 +1,13 @@
 <?xml version="1.0"?>
 <robot xmlns:xacro="http://www.ros.org/wiki/xacro"  name="robot">
+      <xacro:arg name="use_ros2_control" default="true"/>
       <xacro:include filename="robot_core.xacro" />
-      <!-- <xacro:include filename="gazebo_control.xacro" /> -->
+      <xacro:if value="$(arg use_ros2_control)">
+         <xacro:include filename="ros2_control.xacro" />
+      </xacro:if>
+      <xacro:unless value="$(arg use_ros2_control)">
+         <xacro:include filename="gazebo_control.xacro" />
+      </xacro:unless>
       <xacro:include filename="lidar.xacro" />
       <xacro:include filename="camera.xacro" />
-      <xacro:include filename="ros2_control.xacro" />
 </robot>

File: description/robot_core.xacro (robot description, xacro)
@@ -32,5 +32,5 @@
             <box size="0.45 0.40 0.015"/>
         </geometry>
-        <material name="white"/>
+        <material name="black"/>
     </visual>
     <collision>
@@ -49,5 +49,5 @@
 </link>
 <gazebo reference="lower_body">
-    <material>Gazebo/White</material>
+    <material>Gazebo/Black</material>
 </gazebo>
 <!--MIDDLE BODY-->
@@ -62,5 +62,5 @@
             <box size="0.29 0.40 0.14"/>
         </geometry>
-        <material name="white"/>
+        <material name="black"/>
     </visual>
     <collision>
@@ -78,5 +78,5 @@
 </link>
 <gazebo reference="middle_body">
-    <material>Gazebo/White</material>
+    <material>Gazebo/Black</material>
 </gazebo>
 <!--UPPER BODY-->
@@ -91,5 +91,5 @@
             <box size="0.45 0.40 0.015"/>
         </geometry>
-        <material name="white"/>
+        <material name="black"/>
     </visual>
     <collision>
@@ -107,5 +107,5 @@
 </link>
 <gazebo reference="upper_body">
-    <material>Gazebo/White</material>
+    <material>Gazebo/Black</material>
 </gazebo>
 <!--LIDAR MOUNT-->
@@ -120,5 +120,5 @@
             <box size="0.07 0.06 0.05"/>
         </geometry>
-        <material name="black"/>
+        <material name="white"/>
     </visual>
     <collision>
@@ -136,5 +136,5 @@
 </link>
 <gazebo reference="lidar_mount">
-    <material>Gazebo/Black</material>
+    <material>Gazebo/White</material>
 </gazebo>
 <!--front_left_pillar_joint-->
@@ -149,5 +149,5 @@
             <box size="0.03 0.016 0.14"/>
         </geometry>
-        <material name="orange"/>
+        <material name="black"/>
     </visual>
     <collision>
@@ -165,5 +165,5 @@
 </link>
 <gazebo reference="front_left_pillar">
-    <material>Gazebo/Orange</material>
+    <material>Gazebo/Black</material>
 </gazebo>
 <!--front_right_pillar_joint-->
@@ -178,5 +178,5 @@
             <box size="0.03 0.016 0.14"/>
         </geometry>
-        <material name="orange"/>
+        <material name="black"/>
     </visual>
     <collision>
@@ -194,5 +194,5 @@
 </link>
 <gazebo reference="front_right_pillar">
-    <material>Gazebo/Orange</material>
+    <material>Gazebo/Black</material>
 </gazebo>
 <!-- LEFT MOTOR -->
@@ -208,5 +208,5 @@
             <box size="0.14 0.055 0.074"/>
         </geometry>
-        <material name="black"/>
+        <material name="white"/>
     </visual>
     <collision>
@@ -225,5 +225,5 @@
 </link>
 <gazebo reference="left_motor">
-    <material>Gazebo/Black</material>
+    <material>Gazebo/White</material>
 </gazebo>
 <!-- RIGHT MOTOR -->
@@ -239,5 +239,5 @@
             <box size="0.14 0.055 0.074"/>
         </geometry>
-        <material name="black"/>
+        <material name="white"/>
     </visual>
     <collision>
@@ -256,5 +256,5 @@
 </link>
 <gazebo reference="right_motor">
-    <material>Gazebo/Black</material>
+    <material>Gazebo/White</material>
 </gazebo>
 <!-- LEFT WHEEL-->
@@ -339,5 +339,5 @@
 </link>
 <gazebo reference="caster_front_left">
-    <material>Gazebo/orange</material>
+    <material>Gazebo/Orange</material>
     <mu1 value="0.001"/>
     <mu2 value="0.001"/>
@@ -366,5 +366,5 @@
 </link>
 <gazebo reference="caster_front_right">
-    <material>Gazebo/orange</material>
+    <material>Gazebo/Orange</material>
     <mu1 value="0.001"/>
     <mu2 value="0.001"/>
@@ -393,5 +393,5 @@
 </link>
 <gazebo reference="caster_rear_left">
-    <material>Gazebo/orange</material>
+    <material>Gazebo/Orange</material>
     <mu1 value="0.001"/>
     <mu2 value="0.001"/>
@@ -420,5 +420,5 @@
 </link>
 <gazebo reference="caster_rear_right">
-    <material>Gazebo/orange</material>
+    <material>Gazebo/Orange</material>
     <mu1 value="0.001"/>
     <mu2 value="0.001"/>

File: description/ros2_control.xacro (robot description, xacro)
@@ -1,5 +1,33 @@
 <?xml version="1.0"?>
 <robot xmlns:xacro="http://www.ros.org/wiki/xacro">
-    <ros2_control name="GazeboSystem" type="system">
+    <ros2_control name="RealRobot" type="system">
+        <hardware>
+            <plugin>diffdrive_arduino/DiffDriveArduinoHardware</plugin>
+            <param name="left_wheel_name">left_wheel_joint</param>
+            <param name="right_wheel_name">right_wheel_joint</param>
+            <param name="loop_rate">30</param>
+            <param name="device">/dev/ttyACM0</param>
+            <param name="baud_rate">57600</param>
+            <param name="timeout_ms">1000</param>
+            <param name="enc_counts_per_rev">3450</param>
+        </hardware>
+        <joint name="left_wheel_joint">
+            <command_interface name="velocity">
+                <param name="min">-10</param>
+                <param name="max">10</param>
+            </command_interface>
+            <state_interface name="position"/>
+            <state_interface name="velocity"/>
+        </joint>
+        <joint name="right_wheel_joint">
+            <command_interface name="velocity">
+                <param name="min">-10</param>
+                <param name="max">10</param>
+            </command_interface>
+            <state_interface name="position"/>
+            <state_interface name="velocity"/>
+        </joint>
+    </ros2_control>
+        <!-- <ros2_control name="GazeboSystem" type="system">
         <hardware>
             <plugin>gazebo_ros2_control/GazeboSystem</plugin>
@@ -21,5 +49,5 @@
             <state_interface name="position"/>
         </joint>
-    </ros2_control>
+    </ros2_control> -->
     <gazebo>
         <plugin name="gazebo_ros2_control" filename="libgazebo_ros2_control.so">
