Commit message: Created core URDF

File: description/lidar.xacro (robot description, xacro)
@@ -4,5 +4,5 @@
        <parent link="lidar_mount"/>
        <child link="laser_frame"/>
-       <origin xyz="0 0 0.035" rpy="0 0 0"/>
+       <origin xyz="0 0 0.035" rpy="0 0 ${pi}"/>
     </joint>
     <link name="laser_frame">

File: description/robot_core.xacro (robot description, xacro)
@@ -20,9 +20,17 @@
     <link name="base_link">
     </link>
+<!--BASE_FROOTPRINT LINK-->
+    <joint name="base_footprint_joint" type="fixed">
+        <parent link="base_link"/>
+        <child link="base_footprint"/>
+        <origin xyz="0 0 0" rpy="0 0 0"/>
+    </joint>
+    <link name="base_footprint">
+    </link>
 <!-- LOWER BODY -->
 <joint name="lower_body_joint" type="fixed">
     <parent link="base_link"/>
     <child link="lower_body"/>
-    <origin xyz="0 0 0"/>
+    <origin xyz="0 0 0.1"/>
 </joint>
 <link name="lower_body">
@@ -142,5 +150,5 @@
     <parent link="lower_body"/>
     <child link="front_left_pillar"/>
-    <origin xyz="0.18 0.177 0.085"/>
+    <origin xyz="0.15 0.15 0.085"/>
 </joint>
 <link name="front_left_pillar">
@@ -171,5 +179,5 @@
     <parent link="lower_body"/>
     <child link="front_right_pillar"/>
-    <origin xyz="0.18 -0.177 0.085"/>
+    <origin xyz="0.15 -0.15 0.085"/>
 </joint>
 <link name="front_right_pillar">
@@ -262,5 +270,5 @@
     <parent link="base_link"/>
     <child link="left_wheel"/>
-    <origin xyz="0 0.2075 -0.05" rpy="-${pi/2} 0 0"/>
+    <origin xyz="0 0.2075 0.05" rpy="-${pi/2} 0 0"/>
     <axis xyz="0 0 1"/>
 </joint>
@@ -291,5 +299,5 @@
     <parent link="base_link"/>
     <child link="right_wheel"/>
-    <origin xyz="0 -0.2075 -0.05" rpy="${pi/2} 0 0"/>
+    <origin xyz="0 -0.2075 0.05" rpy="${pi/2} 0 0"/>
     <axis xyz="0 0 -1"/>
 </joint>

File: description/ros2_control.xacro (robot description, xacro)
@@ -7,8 +7,8 @@
             <param name="right_wheel_name">right_wheel_joint</param>
             <param name="loop_rate">30</param>
-            <param name="device">/dev/ttyACM0</param>
+            <param name="device">/dev/serial/by-path/platform-fd500000.pcie-pci-0000:01:00.0-usb-0:1.2:1.0</param>
             <param name="baud_rate">57600</param>
             <param name="timeout_ms">1000</param>
-            <param name="enc_counts_per_rev">3450</param>
+            <param name="enc_counts_per_rev">995</param>
         </hardware>
         <joint name="left_wheel_joint">
